Commit message: stuff

File: Urdf/gluon.urdf (robot description, URDF)
Before this commit: robot gluon, 8 links, 7 joints
Links:
- link 1_Link: geometry visual mesh filename=./dae_meshes/1_Link.dae
- link 2_Link: geometry visual mesh filename=./dae_meshes/2_Link.dae
- link 3_Link: geometry visual mesh filename=./dae_meshes/3_Link.dae
- link 4_Link: geometry visual mesh filename=./dae_meshes/4_Link.dae
- link 5_Link: geometry visual mesh filename=./dae_meshes/5_Link.dae
- link 6_Link: geometry visual mesh filename=./dae_meshes/6_Link.dae
- link base_link: geometry visual mesh filename=./dae_meshes/base_link.dae

Commit message: Orientation errors

File: Urdf/gluon.urdf (robot description, URDF)
Before this commit: robot gluon, 8 links, 7 joints
Joints:
- joint axis_joint_1: axis 0 0 -1 -> 0 0 1
- joint axis_joint_2: axis -1 0 0 -> 0 0 1; origin xyz=0.080113 -2.2695E-05 0 rpy=0 0 0 -> xyz=0.080113 -2.2695E-05 0 rpy=0 1.57079632679 0
- joint axis_joint_3: axis 1 0 0 -> 0 0 1; origin xyz=0 0 0.17447 rpy=0 0 0 -> xyz=-0.17447 0 0 rpy=0 0 0
- joint axis_joint_4: axis -1 0 0 -> 0 0 1; origin xyz=-0.084516 0 0.17442 rpy=0 0 0 -> xyz=-0.17442 0 -0.084516 rpy=0 3.14159265358 0
- joint axis_joint_5: origin xyz=0.080113 2.2695E-05 0 rpy=0 0 0 -> xyz=0 2.2695E-05 -0.080113 rpy=0 1.57079632679 0
- joint axis_joint_6: axis -1 0 0 -> 0 0 1; origin xyz=0 -4.5391E-05 0.080089 rpy=0 0 0 -> xyz=0 -4.5391E-05 0.080089 rpy=0 1.57079632679 0
